File: hw/EinkPicFrame.kicad_pcb (KiCad board)
At the start: 2 copper layers, 80 x 21.6 mm, 29 parts, among them J1 SD, J2 AVR-ISP-6, J3 EPD, J4 Power, J7 Debug, Q1 2N7000, Q2 2N7000, SW1 SW_Push, U1 ATmega328P-PU, Y1 Crystal

Commit message: HW: Revert to KiCad 5
I have trouble getting 3d view to work wiht KiCad 6
Other:
- net class Default added: clearance 0.2, trace_width 0.25, via_dia 0.8, via_drill 0.4
- net class Power added: clearance 0.2, trace_width 0.5, via_dia 0.8, via_drill 0.4

Commit message: HW: Ubgrade to KiCad 6.0
Jut open project in Kicad 6 and save to new format.
Other:
- net class Default removed
- net class Power removed
